Commit message: ft sensor: added config but not working yet

File: xacro/go1/gazebo.xacro (robot description, xacro)
@@ -36,23 +36,4 @@
 <!--        </plugin>-->
 <!--    </gazebo>-->
-<!--    <gazebo reference="imu_link">-->
-<!--        <gravity>true</gravity>-->
-<!--        <sensor name="imu_sensor" type="imu">-->
-<!--            <always_on>true</always_on>-->
-<!--            <update_rate>1000</update_rate>-->
-<!--            <visualize>true</visualize>-->
-<!--            <topic>__default_topic__</topic>-->
-<!--            <plugin filename="libgazebo_ros_imu_sensor.so" name="imu_plugin">-->
-<!--                <topicName>trunk_imu</topicName>-->
-<!--                <bodyName>imu_link</bodyName>-->
-<!--                <updateRateHZ>1000.0</updateRateHZ>-->
-<!--                <gaussianNoise>0.0</gaussianNoise>-->
-<!--                <xyzOffset>0 0 0</xyzOffset>-->
-<!--                <rpyOffset>0 0 0</rpyOffset>-->
-<!--                <frameName>imu_link</frameName>-->
-<!--            </plugin>-->
-<!--            <pose>0 0 0 0 0 0</pose>-->
-<!--        </sensor>-->
-<!--    </gazebo>-->
     <!-- Foot contacts. -->
 <!--    <gazebo reference="FR_calf">-->

File: xacro/go1/ros2_control.xacro (robot description, xacro)
@@ -93,4 +93,12 @@
             <state_interface name="linear_acceleration.z"/>
         </sensor>
+        <sensor name="fr_ft_sensor">
+            <state_interface name="force.x"/>
+            <state_interface name="force.y"/>
+            <state_interface name="force.z"/>
+            <state_interface name="torque.x"/>
+            <state_interface name="torque.y"/>
+            <state_interface name="torque.z"/>
+        </sensor>
     </ros2_control>
     <gazebo>
@@ -99,4 +107,5 @@
         </plugin>
         <plugin filename="gz-sim-imu-system" name="gz::sim::systems::Imu"/>
+        <plugin filename="gz-sim-forcetorque-system" name="gz::sim::systems::ForceTorque"/>
     </gazebo>
     <gazebo reference="imu_link">
@@ -162,3 +171,15 @@
         </sensor>
     </gazebo>
+    <gazebo reference="FR_foot_fixed">
+        <sensor name="fr_ft_sensor" type="force_torque">
+            <always_on>1</always_on>
+            <update_rate>500</update_rate>
+            <visualize>true</visualize>
+            <topic>FR_joint/force_torque</topic>
+            <force_torque>
+                <frame>parent</frame>
+                <measure_direction>child_to_parent</measure_direction>
+            </force_torque>
+        </sensor>
+    </gazebo>
 </robot>

File: xacro/go1/transmission.xacro (robot description, xacro)
@@ -32,4 +32,15 @@
             </actuator>
         </transmission>
+        <transmission name="${name}_foot_ft_trans">
+            <type>transmission_interface/SimpleTransmission</type>
+            <joint name="${name}_foot_fixed">
+                <hardwareInterfaces>
+                    <hardwareInterface>hardware_interface/ForceTorqueSensorInterface</hardwareInterface>
+                </hardwareInterfaces>
+            </joint>
+            <actuator name="${name}_foot_ft_actuator">
+                <mechanicalReduction>1</mechanicalReduction>
+            </actuator>
+        </transmission>
     </xacro:macro>
 </robot>

File: xacro/go1/ultrasound.xacro (robot description, xacro)
@@ -2,10 +2,10 @@
 <robot xmlns:xacro="http://www.ros.org/wiki/xacro">
     <xacro:macro name="ultrasound" params="name *origin">
-        <joint name="ultraSound_joint_${name}" type="fixed">
+        <joint name="ultrasound_joint_${name}" type="fixed">
             <xacro:insert_block name="origin"/>
             <parent link="trunk"/>
-            <child link="ultraSound_${name}"/>
+            <child link="ultrasound_${name}"/>
         </joint>
-        <link name="ultraSound_${name}">
+        <link name="ultrasound_${name}">
             <collision>
             <origin xyz="0 0 0" rpy="0 0 0"/>
